File: MicroController/MicroController.kicad_pcb (KiCad board)
At the start: 2 copper layers, 48.3 x 81.3 mm, 14 parts, among them J1 Conn_01x02_Male, J2 Conn_01x02_Male, J3 Conn_01x02_Male, J4 Conn_01x04_Male, U1 MPU6050

Commit message: update
Parts:
- moved J2 12.7 mm to (162.6, 88.9)
- moved J3 10.2 mm to (175.3, 88.9)
Connections:
- J2 pad 2: Net-(J1-Pad2) -> Net-(J1-Pad1)
- J3 pad 1: Net-(J1-Pad1) -> Net-(J2-Pad1)
- J3 pad 2: Net-(J2-Pad1) -> Net-(J1-Pad2)
Routing:
- net Net-(J2-Pad1): track 7.66 -> 17.7 mm
Changed lines of the file:
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@@
     (thickness 1.6)
     (drawings 4)
-    (tracks 41)
+    (tracks 44)
     (zones 0)
     (modules 14)
@@
   )
   (module Connector_JST:JST_XH_B2B-XH-A_1x02_P2.50mm_Vertical (layer F.Cu)
-    (at 175.26 88.9)
+    (at 162.6 88.9)
     (descr "JST XH series connector, B2B-XH-A (http://www.jst-mfg.com/product/pdf/eng/eXH.pdf), generated with kicad-footprint-generator")
     (tags "connector JST XH vertical")
@@
       (net 33 "Net-(J2-Pad1)"))
     (pad 2 thru_hole oval (at 2.5 0) (size 1.7 2) (drill 1) (layers *.Cu *.Mask)
-      (net 32 "Net-(J1-Pad2)"))
+      (net 31 "Net-(J1-Pad1)"))
     (model ${KISYS3DMOD}/Connector_JST.3dshapes/JST_XH_B2B-XH-A_1x02_P2.50mm_Vertical.wrl
       (at (xyz 0 0 0))
@@
   )
   (module Connector_JST:JST_XH_B2B-XH-A_1x02_P2.50mm_Vertical (layer F.Cu)
-    (at 165.1 88.9)
+    (at 175.26 88.9)
     (descr "JST XH series connector, B2B-XH-A (http://www.jst-mfg.com/product/pdf/eng/eXH.pdf), generated with kicad-footprint-generator")
     (tags "connector JST XH vertical")
@@
     (fp_line (start -2.45 -2.35) (end -2.45 3.4) (layer F.Fab) (width 0.1))
     (pad 2 thru_hole oval (at 2.5 0) (size 1.7 2) (drill 1) (layers *.Cu *.Mask)
+      (net 32 "Net-(J1-Pad2)"))
+    (pad 1 thru_hole roundrect (at 0 0) (size 1.7 2) (drill 1) (layers *.Cu *.Mask) (roundrect_rratio 0.147059)
       (net 33 "Net-(J2-Pad1)"))
-    (pad 1 thru_hole roundrect (at 0 0) (size 1.7 2) (drill 1) (layers *.Cu *.Mask) (roundrect_rratio 0.147059)
-      (net 31 "Net-(J1-Pad1)"))
     (model ${KISYS3DMOD}/Connector_JST.3dshapes/JST_XH_B2B-XH-A_1x02_P2.50mm_Vertical.wrl
       (at (xyz 0 0 0))
@@
   (segment (start 160.18 38.1) (end 162.56 38.1) (width 0.25) (layer B.Cu) (net 29))
   (segment (start 160.1 38.02) (end 160.18 38.1) (width 0.25) (layer B.Cu) (net 29))
-  (segment (start 165.1 88.9) (end 165.1 81.28) (width 0.25) (layer B.Cu) (net 31))
   (segment (start 165.1 81.28) (end 177.8 81.28) (width 0.25) (layer B.Cu) (net 31))
   (segment (start 177.8 81.28) (end 177.8 66.04) (width 0.25) (layer B.Cu) (net 31))
   (segment (start 177.8 66.04) (end 177.8 17.78) (width 0.25) (layer B.Cu) (net 31))
+  (segment (start 165.1 88.9) (end 165.1 81.28) (width 0.25) (layer B.Cu) (net 31))
   (segment (start 175.3 17.93) (end 175.26 17.97) (width 0.25) (layer B.Cu) (net 32))
   (segment (start 175.3 17.78) (end 175.3 17.93) (width 0.25) (layer B.Cu) (net 32))
@@
   (segment (start 177.76 83.86) (end 177.76 88.9) (width 0.25) (layer B.Cu) (net 32))
   (segment (start 177.8 83.82) (end 177.76 83.86) (width 0.25) (layer B.Cu) (net 32))
-  (segment (start 167.6 88.9) (end 175.26 88.9) (width 0.25) (layer B.Cu) (net 33))
+  (segment (start 175.26 88.9) (end 175.26 91.44) (width 0.25) (layer B.Cu) (net 33))
+  (segment (start 162.6 88.9) (end 162.6 91.4) (width 0.25) (layer B.Cu) (net 33))
+  (segment (start 162.6 91.4) (end 162.64 91.44) (width 0.25) (layer B.Cu) (net 33))
+  (segment (start 162.64 91.44) (end 175.26 91.44) (width 0.25) (layer B.Cu) (net 33))
 )
