File: MicroController/MicroController.sch (KiCad schematic (older format))
At the start: 6 parts, among them J1 Conn_01x02_Male, J2 Conn_01x02_Male, J3 Conn_01x02_Male, J4 Conn_01x04_Male, U1 MPU6050

Commit message: update
Connections:
- net at J1.1 (Pin_1): now also J2.2 (Pin_2); no longer J3.1 (Pin_1)
- net at J1.2 (Pin_2): now also J3.2 (Pin_2); no longer J2.2 (Pin_2)
- net at J2.1 (Pin_1): now also J3.1 (Pin_1); no longer J3.2 (Pin_2)
Other:
- moved on the sheet: J2
Changed lines of the file:
@@
 	1    0    0    -1
 $EndComp
-Wire Wire Line
-	4650 4850 4800 4850
-Wire Wire Line
-	4800 5250 4650 5250
 NoConn ~ 3050 4000
 NoConn ~ 3050 3900
@@
 L Connector:Conn_01x02_Male J2
 U 1 1 5E1309D5
-P 5200 5200
-F 0 "J2" H 5172 5082 50  0000 R CNN
-F 1 "Conn_01x02_Male" H 5172 5173 50  0000 R CNN
-F 2 "Connector_JST:JST_XH_B2B-XH-A_1x02_P2.50mm_Vertical" H 5200 5200 50  0001 C CNN
-F 3 "~" H 5200 5200 50  0001 C CNN
-	1    5200 5200
+P 5300 5100
+F 0 "J2" H 5272 4982 50  0000 R CNN
+F 1 "Conn_01x02_Male" H 5272 5073 50  0000 R CNN
+F 2 "Connector_JST:JST_XH_B2B-XH-A_1x02_P2.50mm_Vertical" H 5300 5100 50  0001 C CNN
+F 3 "~" H 5300 5100 50  0001 C CNN
+	1    5300 5100
 	-1   0    0    1
 $EndComp
-Wire Wire Line
-	4800 4850 4800 5250
-Wire Wire Line
-	5000 4950 5000 5100
-Wire Wire Line
-	4650 4950 5000 4950
-Wire Wire Line
-	5000 5200 5000 5350
-Wire Wire Line
-	4650 5350 5000 5350
 Text GLabel 3050 3500 0    50   Input ~ 0
 SDA
@@
 Text GLabel 3050 4300 0    50   Input ~ 0
 LED_G
+Wire Wire Line
+	4650 4850 5100 4850
+Wire Wire Line
+	5100 4850 5100 5000
+Wire Wire Line
+	5100 5100 5100 5250
+Wire Wire Line
+	5100 5250 4650 5250
+Wire Wire Line
+	4650 4950 4750 4950
+Wire Wire Line
+	4750 4950 4750 5350
+Wire Wire Line
+	4750 5350 4650 5350
 $EndSCHEMATC
